File: fc2.1/untitled.brd (EAGLE design)
At the start: 64 x 43.4 mm, 60 parts, among them CON1 XT30UPB-M, IC1 TC1264-3.3VDBTR, IC2 BMI088, IC3 FT231XS-R, IC5 L7805CDT-TR, J1 503398-1892, Q1 SISH536DN-T1-GE3, Q2 SISH536DN-T1-GE3, Q5 SISH536DN-T1-GE3, U1 RP2040

Commit message: Add files via upload
Parts:
- moved R12 0.67 mm to (22.5, 25.8)
Connections:
- removed net N$12: IC3.16, IC3.6
- net 3.3V: now also IC3.14, J2.3
- net 5V: no longer J2.3
- net GND: now also IC3.16, IC3.6
- net SD_DETECT: now also U1.32; no longer U1.37
Routing:
- net GND: track 103.1 -> 123.5 mm, vias 14 -> 21
- net 5V: track 173.7 -> 158.2 mm
- net VIN: track 99.3 -> 91.4 mm
- net MOSI: track 81.1 -> 88.9 mm
- net N$12: track 5.70 -> 0.00 mm
- net N$19: track 43.3 -> 47.9 mm
- net N$7: track 70.5 -> 72.6 mm
- net QSPI_SD3: track 24.8 -> 26.5 mm
- net SD_DETECT: track 38.1 -> 36.4 mm
- net RXE: track 74.8 -> 76.3 mm
- net SCK: track 77.9 -> 79.2 mm
- net 3.3V: track 123.3 -> 124.5 mm
- net SCL: track 137.7 -> 139.0 mm
- net N$5: track 32.0 -> 32.6 mm
- net N$25: track 22.0 -> 21.4 mm
