File: fc2.1/untitled.sch (EAGLE design)
At the start: 58 parts, among them CON1 XT30UPB-M, IC1 TC1264-3.3VDBTR, IC2 BMI088, IC3 FT231XS-R, IC5 L7805CDT-TR, J1 503398-1892, Q1 SISH536DN-T1-GE3, Q2 SISH536DN-T1-GE3, Q5 SISH536DN-T1-GE3, U1 RP2040

Commit message: Add files via upload
Connections:
- removed net N$12: IC3.GND_1, IC3.GND_2
- net 3.3V: now also IC3.RESET#, J2.3
- net 5V: no longer J2.3
- net GND: now also IC3.GND_1, IC3.GND_2
- net SD_DETECT: now also U1.GPIO21; no longer U1.GPIO25
Changed lines of the file:
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@@
 <setting verticaltext="up"/>
 </settings>
-<grid distance="0.1" unitdist="inch" unit="inch" style="lines" multiple="1" display="no" altdistance="0.01" altunitdist="inch" altunit="inch"/>
+<grid distance="0.05" unitdist="inch" unit="inch" style="lines" multiple="1" display="no" altdistance="0.01" altunitdist="inch" altunit="inch"/>
 <layers>
 <layer number="1" name="Top" color="4" fill="1" visible="no" active="no"/>
@@
 <label x="5.08" y="83.82" size="1.778" layer="95"/>
 </segment>
+<segment>
+<pinref part="IC3" gate="G$1" pin="GND_1"/>
+<wire x1="297.18" y1="43.18" x2="297.18" y2="40.64" width="0.1524" layer="91"/>
+<pinref part="IC3" gate="G$1" pin="GND_2"/>
+<wire x1="297.18" y1="40.64" x2="297.18" y2="30.48" width="0.1524" layer="91"/>
+<wire x1="299.72" y1="43.18" x2="299.72" y2="40.64" width="0.1524" layer="91"/>
+<wire x1="299.72" y1="40.64" x2="297.18" y2="40.64" width="0.1524" layer="91"/>
+<junction x="297.18" y="40.64"/>
+<label x="297.18" y="35.56" size="1.778" layer="95"/>
+</segment>
 </net>
 <net name="QSPI_SD0" class="0">
@@
 <wire x1="274.32" y1="91.44" x2="274.32" y2="111.76" width="0.1524" layer="91"/>
 <wire x1="274.32" y1="111.76" x2="297.18" y2="111.76" width="0.1524" layer="91"/>
+<pinref part="IC3" gate="G$1" pin="RESET#"/>
+<wire x1="281.94" y1="78.74" x2="266.7" y2="78.74" width="0.1524" layer="91"/>
+<wire x1="266.7" y1="78.74" x2="266.7" y2="91.44" width="0.1524" layer="91"/>
+<wire x1="266.7" y1="91.44" x2="274.32" y2="91.44" width="0.1524" layer="91"/>
+<junction x="274.32" y="91.44"/>
 </segment>
 <segment>
@@
 <wire x1="354.33" y1="-85.09" x2="378.46" y2="-85.09" width="0.1524" layer="91"/>
 <label x="370.84" y="-85.09" size="1.778" layer="95"/>
+</segment>
+<segment>
+<pinref part="J2" gate="G$1" pin="3"/>
+<wire x1="208.28" y1="-57.15" x2="233.68" y2="-57.15" width="0.1524" layer="91"/>
+<label x="213.36" y="-57.15" size="1.778" layer="95"/>
 </segment>
 </net>
@@
 <label x="161.29" y="-57.15" size="1.778" layer="95"/>
 </segment>
-<segment>
-<pinref part="J2" gate="G$1" pin="3"/>
-<wire x1="208.28" y1="-57.15" x2="233.68" y2="-57.15" width="0.1524" layer="91"/>
-<label x="213.36" y="-57.15" size="1.778" layer="95"/>
-</segment>
 </net>
 <net name="USBD+" class="0">
@@
 <pinref part="ESP_PROG" gate="G$1" pin="NO_2"/>
 <wire x1="257.81" y1="182.88" x2="261.62" y2="182.88" width="0.1524" layer="91"/>
-</segment>
-</net>
-<net name="N$12" class="0">
-<segment>
-<pinref part="IC3" gate="G$1" pin="GND_1"/>
-<wire x1="297.18" y1="43.18" x2="297.18" y2="40.64" width="0.1524" layer="91"/>
-<pinref part="IC3" gate="G$1" pin="GND_2"/>
-<wire x1="297.18" y1="40.64" x2="297.18" y2="30.48" width="0.1524" layer="91"/>
-<wire x1="299.72" y1="43.18" x2="299.72" y2="40.64" width="0.1524" layer="91"/>
-<wire x1="299.72" y1="40.64" x2="297.18" y2="40.64" width="0.1524" layer="91"/>
-<junction x="297.18" y="40.64"/>
 </segment>
 </net>
@@
 </segment>
 <segment>
-<pinref part="U1" gate="U1" pin="GPIO25"/>
-<wire x1="60.96" y1="17.78" x2="82.55" y2="17.78" width="0.1524" layer="91"/>
-<label x="64.77" y="17.78" size="1.778" layer="95"/>
-</segment>
-</net>
+<pinref part="U1" gate="U1" pin="GPIO21"/>
+<wire x1="60.96" y1="27.94" x2="82.55" y2="27.94" width="0.1524" layer="91"/>
+<label x="64.77" y="27.94" size="1.778" layer="95"/>
+</segment>
+</net>
